File: _Fluxamasynth32/Fluxamasynth32.brd (EAGLE design)
At the start: 52.9 x 48.9 mm, 52 parts, among them J1 POWER_JACKSLT, U1 ESP-WROOM-03, U2 V_REG_317SMD

Commit message: Feather, Pi updates
Connections:
- net +3V3: now also U2.4
Routing:
- net GND: track 262.9 -> 273.0 mm
- removed copper zone on layer 16, net +3V3
Other:
- board text added: "/Users/as220/_FluxamasynthGithub/_Fluxamasynth32/Artwork/FLUXYNTHbOTTOMsILK.bmp"
