File: _FluxamasynthPi/FluxamasynthPi.brd (EAGLE design)
At the start: 65 x 30 mm, 41 parts, among them U1 V_REG_LDOSMD

Commit message: Feather, Pi updates
Parts:
- removed C11: 10uf, ModernDevice:C0805K
- removed U1: V_REG_LDOSMD, ModernDevice:SOT23-5
- added MIC_JACK1: (no value), ModernDevice:1X02
Connections:
- removed net +5V: C11.1, U$1.2, U1.1, U1.3
- net +3V3: now also MIC_JACK1.2, U$1.1; no longer U1.5
- net GND: now also MIC_JACK1.1; no longer C11.2, U1.2
Routing:
- net +5V: track 53.3 -> 0.00 mm, vias 1 -> 0
- net +3V3: track 91.4 -> 133.9 mm, vias 0 -> 1
- net GND: track 158.6 -> 156.4 mm
- net N$12: track 6.08 -> 5.37 mm
