File: _FluxamasynthPi/FluxamasynthPi.sch (EAGLE design)
At the start: 41 parts, among them U1 V_REG_LDOSMD

Commit message: Feather, Pi updates
Parts:
- removed C11: 10uf, ModernDevice:C-USC0805K
- removed U1: V_REG_LDOSMD, ModernDevice:V_REG_LDOSMD
- added MIC_JACK1: (no value), ModernDevice:M02PTH
Connections:
- removed net +5V: C11.1, U$1.5V0@1, U1.EN, U1.IN
- net +3V3: now also MIC_JACK1.2, U$1.3V3@1; no longer U1.OUT
- net GND: now also MIC_JACK1.1; no longer C11.2, U1.GND
Other:
- note added: "Fluxamasynth Pi"
